Commit message: modified:   config/nav2_params.yaml 	modified:   src/robot_description/urdf/tracked_robot.urdf

File: src/robot_description/urdf/tracked_robot.urdf (robot description, URDF)
Before this commit: robot tracked_robot, 7 links, 6 joints
Joints:
- joint lidar_joint: origin xyz=0.11 -0.06 0.065 rpy=0 0 0 -> xyz=0.0 -0.06 0.065 rpy=0 0 0

Commit message: Changes to be committed: 	modified:   src/robot_bringup/launch/minimal_all.launch.py 	modified:   src/robot_description/urdf/tracked_robot.urdf 	modified:   src/robot_gz/models/tracked_robot/model.sdf 	modified:   src/robot_gz/worlds/tracked_robot_world.sdf 	modified:   src/robot_sim_control/package.xml 	new file:   src/robot_sim_control/robot_sim_control/robotarm_gui.py 	modified:   src/robot_sim_control/setup.py

File: src/robot_description/urdf/tracked_robot.urdf (robot description, URDF)
Before this commit: robot tracked_robot, 23 links, 22 joints
Links:
- added link Robotarm, mass 0.05; visual cylinder length=0.2 radius=0.01
- added link gripper_plate, mass 0.0001; collision box size=0.02 0.14 0.06; visual box size=0.02 0.14 0.06
- added link leadscrew, mass 0.0; visual cylinder length=0.2 radius=0.01
- added link left_gripper_finger, mass 0.02; collision box size=0.12 0.015 0.04; visual box size=0.12 0.015 0.04
- added link right_gripper_finger, mass 0.02; collision box size=0.12 0.015 0.04; visual box size=0.12 0.015 0.04
- added link x_carriage, mass 0.0001
- link ML: geometry visual mesh filename=package://robot_description/meshes/ML.stl scale=0.001 0.001 0.001
- link MR: geometry visual mesh filename=package://robot_description/meshes/MR.stl scale=0.001 0.001 0.001
- link SLOTLBI: geometry visual mesh filename=package://robot_description/meshes/SLOTLBI.stl scale=0.001 0.001 0.001
- link SLOTLFI: geometry visual mesh filename=package://robot_description/meshes/SLOTLFI.stl scale=0.001 0.001 0.001
- link SLOTRFI: geometry visual mesh filename=package://robot_description/meshes/SLOTRFI.stl scale=0.001 0.001 0.001
- link Stepper-1: geometry visual mesh filename=package://robot_description/meshes/Stepper-1.stl scale=0.001 0.001 0.001
- link camera_link: geometry visual mesh filename=package://robot_description/meshes/Camera.stl scale=0.001 0.001 0.001
- link imu_link: geometry visual mesh filename=package://robot_description/meshes/IMU.stl scale=0.001 0.001 0.001
- link lidar_link: geometry visual mesh filename=package://robot_description/meshes/Lidar.stl scale=0.001 0.001 0.001
Joints:
- added joint leadscrew_to_base_link: type fixed, parent base_link, child leadscrew, origin xyz=0.05 0.0 0.15 rpy=0.0 0.0 0.0
- added joint left_gripper_finger_joint: type revolute, parent gripper_plate, child left_gripper_finger, origin xyz=0.0 0.0625 0.0 rpy=0 0 0, axis 0 0 1, limit lower=-0.785 upper=0.785 effort=10 velocity=1.0
- added joint plate_arm_link: type fixed, parent Robotarm, child gripper_plate, origin xyz=0.1 0.0 -0.06 rpy=0 0 0
- added joint right_gripper_finger_joint: type revolute, parent gripper_plate, child right_gripper_finger, origin xyz=0.0 -0.0625 0.0 rpy=0 0 0, axis 0 0 1, limit lower=-0.785 upper=0.785 effort=10 velocity=1.0
- added joint robotarm_x_joint: type prismatic, parent base_link, child x_carriage, origin xyz=0.05 0.0 0.05 rpy=0 0 0, axis 1 0 0, limit lower=-0.2 upper=0.2 effort=100 velocity=0.2
- added joint robotarm_z_joint: type prismatic, parent x_carriage, child Robotarm, origin xyz=0.0 0.0 0.0 rpy=0 0 0, axis 0 0 1, limit lower=1.0 upper=1.0 effort=100 velocity=0.2
- joint left_wheel_joint: type continuous -> fixed
- joint right_wheel_joint: type continuous -> fixed

Commit message: new file:   src/mekk4_bringup/mekk4_bringup/robotarm_safety_node.py 	modified:   src/mekk4_bringup/mekk4_bringup/teddy_approach_node.py 	new file:   src/mekk4_bringup/mekk4_bringup/teddy_grab_node.py 	modified:   src/mekk4_bringup/setup.py 	modified:   src/robot_bringup/launch/minimal_all.launch.py 	modified:   src/robot_bringup/launch/pi_robot.launch.py 	modified:   src/robot_description/urdf/tracked_robot.urdf 	modified:   src/robot_gz/models/tracked_robot/model.sdf 	modified:   src/robot_sim_control/package.xml 	modified:   src/robot_sim_control/robot_sim_control/robotarm_gui.py

File: src/robot_description/urdf/tracked_robot.urdf (robot description, URDF)
Before this commit: robot tracked_robot, 29 links, 28 joints
Joints:
- joint plate_arm_link: origin xyz=0.1 0.0 -0.06 rpy=0 0 0 -> xyz=0.1 0.0 -0.09 rpy=0 0 0
- joint robotarm_x_joint: limit lower=-0.2 upper=0.2 effort=100 velocity=0.2 -> lower=-0.2 upper=0.2 effort=100 velocity=0.01
- joint robotarm_z_joint: limit lower=1.0 upper=1.0 effort=100 velocity=0.2 -> lower=1.0 upper=1.0 effort=100 velocity=0.01
